Commit message: urdf done v:0

File: urdf/robot.urdf.xacro (robot description, xacro)
@@ -28,4 +28,5 @@
     <link name="base_link"></link>
     <joint name="baseLink_chassis" type="fixed">
+        <origin xyz="0.0 0.0 0.36" rpy="0.0 0.0 0.0"/>
         <parent link="base_link" />
         <child link="chassis" />
@@ -33,8 +34,9 @@
     <link name="chassis">
         <xacro:solid_cuboid_inertial width="${chassis_length}" depth="${chassis_width}" height="${chassis_height*20}" mass="${chassis_mass}">
-            <origin xyz="0 -0.266 0.48" />
+            <!-- <origin xyz="0 -0.266 0.48" /> -->
+            <origin xyz="0.0 0.0 0.0" rpy="0.0 0.0 0.0"/>
         </xacro:solid_cuboid_inertial>
         <visual>
-            <origin xyz="0.0 0.0 0.0" rpy="0.0 0.0 0.0" />
+            <origin xyz="0.0 0.0 0.0" rpy="0.0 0.0 0.0"/>
             <geometry>
                 <box size="${chassis_length} ${chassis_width-0.3} ${chassis_height}" />
@@ -42,5 +44,5 @@
         </visual>
         <collision>
-            <origin xyz="0.0 0.0 0.0" rpy="0.0 0.0 0.0" />
+            <origin xyz="0.0 0.0 0.0" rpy="0.0 0.0 0.0"/>
             <geometry>
                 <box size="${chassis_length} ${chassis_width-0.3} ${chassis_height}" />
@@ -48,5 +50,5 @@
         </collision>
     </link>
-    <link name="steering_wheel">
+    <!-- <link name="steering_wheel">
         <inertial>
             <origin xyz="0.0 0.0 0.0" rpy="0.0 0.0 0.0" />
@@ -70,23 +72,23 @@
             </geometry>
         </collision>
-    </link>
+    </link> -->
     <link name="front_left_wheel">
         <inertial>
-            <origin xyz="0.0 0.0 0.0" rpy="0.0 0.0 0.0" />
-            <mass value="7.0" />
-            <inertia ixx="0.586312" ixy="0.0" ixz="0.0" iyy="0.335529" iyz="0.0" izz="0.335529" />
-        </inertial>
-        <visual name="">
-            <origin xyz="0.0 0.0 0.0" rpy="0.0 0.0 0.0" />
-            <geometry>
-                <cylinder radius="${tire_dia / 2}" length="${tire_width}" />
-            </geometry>
-            <material name="">
-                <color rgba="1.0 0.0 0.0 1.0" />
-                <texture filename="" />
-            </material>
-        </visual>
-        <collision>
-            <origin xyz="0.0 0.0 0.0" rpy="0.0 0.0 0.0" />
+            <origin xyz="0.0 0.0 0.0" rpy="-1.57 0.0 0.0" />
+            <mass value="7.0" />
+            <inertia ixx="0.586312" ixy="0.0" ixz="0.0" iyy="0.335529" iyz="0.0" izz="0.335529" />
+        </inertial>
+        <visual name="">
+            <origin xyz="0.0 0.0 0.0" rpy="-1.57 0.0 0.0" />
+            <geometry>
+                <cylinder radius="${tire_dia / 2}" length="${tire_width}" />
+            </geometry>
+            <material name="">
+                <color rgba="1.0 0.0 0.0 1.0" />
+                <texture filename="" />
+            </material>
+        </visual>
+        <collision>
+            <origin xyz="0.0 0.0 0.0" rpy="-1.57 0.0 0.0"/>
             <geometry>
                 <cylinder radius="${tire_dia / 2}" length="${tire_width}" />
@@ -96,20 +98,20 @@
     <link name="front_right_wheel">
         <inertial>
-            <origin xyz="0.0 0.0 0.0" rpy="0.0 0.0 0.0" />
-            <mass value="7.0" />
-            <inertia ixx="0.586312" ixy="0.0" ixz="0.0" iyy="0.335529" iyz="0.0" izz="0.335529" />
-        </inertial>
-        <visual name="">
-            <origin xyz="0.0 0.0 0.0" rpy="0.0 0.0 0.0" />
-            <geometry>
-                <cylinder radius="${tire_dia / 2}" length="${tire_width}" />
-            </geometry>
-            <material name="">
-                <color rgba="1.0 0.0 0.0 1.0" />
-                <texture filename="" />
-            </material>
-        </visual>
-        <collision>
-            <origin xyz="0.0 0.0 0.0" rpy="0.0 0.0 0.0" />
+            <origin xyz="0.0 0.0 0.0" rpy="-1.57 0.0 0.0"/>
+            <mass value="7.0" />
+            <inertia ixx="0.586312" ixy="0.0" ixz="0.0" iyy="0.335529" iyz="0.0" izz="0.335529" />
+        </inertial>
+        <visual name="">
+            <origin xyz="0.0 0.0 0.0" rpy="-1.57 0.0 0.0"/>
+            <geometry>
+                <cylinder radius="${tire_dia / 2}" length="${tire_width}" />
+            </geometry>
+            <material name="">
+                <color rgba="1.0 0.0 0.0 1.0" />
+                <texture filename="" />
+            </material>
+        </visual>
+        <collision>
+            <origin xyz="0.0 0.0 0.0" rpy="-1.57 0.0 0.0" />
             <geometry>
                 <cylinder radius="${tire_dia / 2}" length="${tire_width}" />
@@ -119,20 +121,20 @@
     <link name="rear_left_wheel">
         <inertial>
-            <origin xyz="0.0 0.0 0.0" rpy="0.0 0.0 0.0" />
-            <mass value="7.0" />
-            <inertia ixx="0.586312" ixy="0.0" ixz="0.0" iyy="0.335529" iyz="0.0" izz="0.335529" />
-        </inertial>
-        <visual name="">
-            <origin xyz="0.0 0.0 0.0" rpy="0.0 0.0 0.0" />
-            <geometry>
-                <cylinder radius="${tire_dia / 2}" length="${tire_width}" />
-            </geometry>
-            <material name="">
-                <color rgba="1.0 0.0 0.0 1.0" />
-                <texture filename="" />
-            </material>
-        </visual>
-        <collision>
-            <origin xyz="0.0 0.0 0.0" rpy="0.0 0.0 0.0" />
+            <origin xyz="0.0 0.0 0.0" rpy="1.57 0.0 0.0" />
+            <mass value="7.0" />
+            <inertia ixx="0.586312" ixy="0.0" ixz="0.0" iyy="0.335529" iyz="0.0" izz="0.335529" />
+        </inertial>
+        <visual name="">
+            <origin xyz="0.0 0.0 0.0" rpy="1.57 0.0 0.0" />
+            <geometry>
+                <cylinder radius="${tire_dia / 2}" length="${tire_width}" />
+            </geometry>
+            <material name="">
+                <color rgba="1.0 0.0 0.0 1.0" />
+                <texture filename="" />
+            </material>
+        </visual>
+        <collision>
+            <origin xyz="0.0 0.0 0.0" rpy="1.57 0.0 0.0" />
             <geometry>
                 <cylinder radius="${tire_dia / 2}" length="${tire_width}" />
@@ -142,20 +144,20 @@
     <link name="rear_right_wheel">
         <inertial>
-            <origin xyz="0.0 0.0 0.0" rpy="0.0 0.0 0.0" />
-            <mass value="7.0" />
-            <inertia ixx="0.586312" ixy="0.0" ixz="0.0" iyy="0.335529" iyz="0.0" izz="0.335529" />
-        </inertial>
-        <visual name="">
-            <origin xyz="0.0 0.0 0.0" rpy="0.0 0.0 0.0" />
-            <geometry>
-                <cylinder radius="${tire_dia / 2}" length="${tire_width}" />
-            </geometry>
-            <material name="">
-                <color rgba="1.0 0.0 0.0 1.0" />
-                <texture filename="" />
-            </material>
-        </visual>
-        <collision>
-            <origin xyz="0.0 0.0 0.0" rpy="0.0 0.0 0.0" />
+            <origin xyz="0.0 0.0 0.0" rpy="1.57 0.0 0.0" />
+            <mass value="7.0" />
+            <inertia ixx="0.586312" ixy="0.0" ixz="0.0" iyy="0.335529" iyz="0.0" izz="0.335529" />
+        </inertial>
+        <visual name="">
+            <origin xyz="0.0 0.0 0.0" rpy="1.57 0.0 0.0" />
+            <geometry>
+                <cylinder radius="${tire_dia / 2}" length="${tire_width}" />
+            </geometry>
+            <material name="">
+                <color rgba="1.0 0.0 0.0 1.0" />
+                <texture filename="" />
+            </material>
+        </visual>
+        <collision>
+            <origin xyz="0.0 0.0 0.0" rpy="1.57 0.0 0.0" />
             <geometry>
                 <cylinder radius="${tire_dia / 2}" length="${tire_width}" />
@@ -165,22 +167,22 @@
     <link name="rear_axle">
         <inertial>
-            <origin xyz="0.0 0.0 0.0" rpy="0.0 0.0 0.0"/>
+            <origin xyz="0 0 0" rpy="-1.57 0.0 0.0" />
             <mass value="30.0"/>
             <inertia ixx="0.084375" ixy="0.0" ixz="0.0" iyy="4.64581" iyz="0.0" izz="4.64581"/>
         </inertial>
         <visual name="">
-            <origin xyz="0.0 0.0 0.0" rpy="0.0 0.0 0.0"/>
-            <geometry>
-                <cylinder radius="0.075" length="1.357"/>
-            </geometry>
-            <material name="">
+            <origin xyz="0 0 0" rpy="-1.57 0.0 0.0" />
+            <geometry>
+                <cylinder radius="0.05" length="1.079600"/>
+            </geometry>
+            <!-- <material name="">
                 <color rgba="1.0 0.0 0.0 1.0"/>
                 <texture filename=""/>
-            </material>
-        </visual>
-        <collision>
-            <origin xyz="0.0 0.0 0.0" rpy="0.0 0.0 0.0"/>
-            <geometry>
-                <cylinder radius="0.075" length="1.357"/>
+            </material> -->
+        </visual>
+        <collision>
+            <origin xyz="0 0 0" rpy="-1.57 0.0 0.0" />
+            <geometry>
+                <cylinder radius="0.05" length="1.079600"/>
             </geometry>
         </collision>
@@ -188,12 +190,13 @@
     <link name="front_left_axle">
         <inertial>
-            <origin xyz="0.0 0.0 0.0" rpy="0.0 0.0 0.0"/>
+            <!-- <origin xyz="0.0 -0.38 0.0" rpy="0.0 0.0 0.0" /> -->
             <mass value="0.0"/>
-            <inertia ixx="0.0" ixy="0.0" ixz="0.0" iyy="0.0" iyz="0.0" izz="0.0"/>
-        </inertial>
-        <visual name="">
-            <origin xyz="0.0 0.0 0.0" rpy="0.0 0.0 0.0"/>
-            <geometry>
-                <cylinder radius="0.075" length="1.357"/>
+            <inertia ixx="0.01" ixy="0.0" ixz="0.0" iyy="0.01" iyz="0.0" izz="0.01"/>
+        </inertial>
+        <visual name="">
+            <origin xyz="0.0 0.0 0.0" rpy="0.0 0.0 0.0" />
+            <geometry>
+                <!-- <cylinder radius="0.075" length="1.357"/> -->
+                <sphere radius="0.07"/>
             </geometry>
             <material name="">
@@ -203,7 +206,8 @@
         </visual>
         <collision>
-            <origin xyz="0.0 0.0 0.0" rpy="0.0 0.0 0.0"/>
-            <geometry>
-                <cylinder radius="0.075" length="1.357"/>
+            <origin xyz="0.0 0.0 0.0" rpy="0.0 0.0 0.0" />
+            <geometry>
+                <!-- <cylinder radius="0.075" length="1.357"/> -->
+                <sphere radius="0.07"/>
             </geometry>
         </collision>
@@ -211,12 +215,13 @@
     <link name="front_right_axle">
         <inertial>
-            <origin xyz="0.0 0.0 0.0" rpy="0.0 0.0 0.0"/>
+            <origin xyz="0.0 0.0 0.0" rpy="0.0 0.0 0.0" />
             <mass value="0.0"/>
-            <inertia ixx="0.0" ixy="0.0" ixz="0.0" iyy="0.0" iyz="0.0" izz="0.0"/>
-        </inertial>
-        <visual name="">
-            <origin xyz="0.0 0.0 0.0" rpy="0.0 0.0 0.0"/>
-            <geometry>
-                <cylinder radius="0.075" length="1.357"/>
+            <inertia ixx="0.01" ixy="0.0" ixz="0.0" iyy="0.01" iyz="0.0" izz="0.01"/>
+        </inertial>
+        <visual name="">
+            <!-- <origin xyz="0.0 -0.38 0.0" rpy="0.0 0.0 0.0" /> -->
+            <geometry>
+                <!-- <cylinder radius="0.075" length="1.357"/> -->
+                <sphere radius="0.07"/>
             </geometry>
             <material name="">
@@ -226,12 +231,13 @@
         </visual>
         <collision>
-            <origin xyz="0.0 0.0 0.0" rpy="0.0 0.0 0.0"/>
-            <geometry>
-                <cylinder radius="0.075" length="1.357"/>
+            <!-- <origin xyz="0.0 -0.38 0.0" rpy="0.0 0.0 0.0" /> -->
+            <geometry>
+                <!-- <cylinder radius="0.075" length="1.357"/> -->
+                <sphere radius="0.07"/>
             </geometry>
         </collision>
     </link>
     <!-- joints -->
-    <joint name="steering_wheel_joint" type="revolute">
+    <!-- <joint name="steering_wheel_joint" type="revolute">
         <origin xyz="0.0 0.0 0.0" rpy="0.0 0.0 0.0"/>
         <parent link="chassis"/>
@@ -239,28 +245,26 @@
         <axis xyz="0.0 0.0 0.0"/>
         <limit lower="0.0" upper="0.0" effort="0.0" velocity="0.0"/>
-    </joint>
+    </joint> -->
     <joint name="front_right_axle_joint" type="revolute">
-        <!-- <origin xyz="0.0 0.0 0.0" rpy="0.0 0.0 0.0"/> -->
-        <origin rpy="${degrees_90} 0 0" />
+        <origin xyz="1.0 -0.6 0" rpy="0 0 0" />
         <parent link="chassis"/>
         <child link="front_right_axle"/>
-        <axis xyz="0.0 1.0 0.0"/>
-        <limit lower="0.0" upper="0.0" effort="0.0" velocity="0.0"/>
+        <axis xyz="0.0 0.0 1.0"/>
+        <limit lower="${-degrees_30}" upper="${degrees_30}" effort="${servo_stall_torque}" velocity="${servo_no_load_speed}" />
     </joint>
     <joint name="front_left_axle_joint" type="revolute">
-        <!-- <origin xyz="0.0 0.0 0.0" rpy="0.0 0.0 0.0"/> -->
-        <origin rpy="${degrees_90} 0 0" />
+        <origin xyz="1.0 0.6 0" rpy="0 0 0" />
         <parent link="chassis"/>
         <child link="front_left_axle"/>
-        <axis xyz="0.0 1.0 0.0"/>
-        <limit lower="0.0" upper="0.0" effort="0.0" velocity="0.0"/>
-    </joint>
-    <joint name="rear_axle_joint" type="revolute">
-        <!-- <origin xyz="0.0 0.0 0.0" rpy="0.0 0.0 0.0"/> -->
-        <origin rpy="${degrees_90} 0 0" />
+        <axis xyz="0.0 0 1.0"/>
+        <limit lower="${-degrees_30}" upper="${degrees_30}" effort="${servo_stall_torque}" velocity="${servo_no_load_speed}" />
+    </joint>
+    <joint name="rear_axle_joint" type="fixed">
+        <origin xyz="-1.0 0.0 0" rpy="0 0.0 0.0"/>
+        <!-- <origin rpy="${degrees_90} 0 0" /> -->
         <parent link="chassis"/>
         <child link="rear_axle"/>
-        <axis xyz="0.0 1.0 0.0"/>
-        <limit lower="0.0" upper="0.0" effort="0.0" velocity="0.0"/>
+        <!-- <axis xyz="0.0 1.0 0.0"/> -->
+        <!-- <limit lower="0.0" upper="0.0" effort="0.0" velocity="0.0"/> -->
     </joint>
     <joint name="front_right_wheel_joint" type="revolute">
@@ -268,5 +272,5 @@
         <parent link="front_right_axle"/>
         <child link="front_right_wheel"/>
-        <axis xyz="0 0 1" />
+        <axis xyz="0 1 0" />
         <limit lower="${-degrees_30}" upper="${degrees_30}" effort="${servo_stall_torque}" velocity="${servo_no_load_speed}" />
     </joint>
@@ -275,19 +279,19 @@
         <parent link="front_left_axle"/>
         <child link="front_left_wheel"/>
-        <axis xyz="0 0 1" />
+        <axis xyz="0 1 0" />
         <limit lower="${-degrees_30}" upper="${degrees_30}" effort="${servo_stall_torque}" velocity="${servo_no_load_speed}" />
     </joint>
     <joint name="rear_right_wheel_joint" type="revolute">
-        <origin xyz="0.0 0.0 0.0" rpy="0.0 0.0 0.0"/>
+        <origin xyz="0 -0.6 0.0" rpy="0.0 0.0 0.0"/>
         <parent link="rear_axle"/>
         <child link="rear_right_wheel"/>
-        <axis xyz="0 0 1" />
+        <axis xyz="0 1 0" />
         <limit lower="${-degrees_30}" upper="${degrees_30}" effort="${servo_stall_torque}" velocity="${servo_no_load_speed}" />
     </joint>
     <joint name="rear_left_wheel_joint" type="revolute">
-        <origin xyz="0.0 0.0 0.0" rpy="0.0 0.0 0.0"/>
+        <origin xyz="0 0.6 0.0" rpy="0.0 0.0 0.0"/>
         <parent link="rear_axle"/>
         <child link="rear_left_wheel"/>
-        <axis xyz="0 0 1" />
+        <axis xyz="0 1 0" />
         <limit lower="${-degrees_30}" upper="${degrees_30}" effort="${servo_stall_torque}" velocity="${servo_no_load_speed}" />
     </joint>

Commit message: update gazebo

File: urdf/robot.urdf.xacro (robot description, xacro)
@@ -1,4 +1,6 @@
 <?xml version="1.0"?>
 <robot name="astrid" xmlns:xacro="http://www.ros.org/wiki/xacro">
+    <xacro:include filename="$(find astrid-simulation)/urdf/common_properties.xacro"/>
+    <xacro:include filename="$(find astrid-simulation)/urdf/astrid.gazebo.xacro"/>
     <!-- Degree-to-radian conversions -->
     <xacro:property name="degrees_45" value="0.785398163" />
@@ -26,4 +28,10 @@
     <xacro:property name="servo_stall_torque" value="57" />
     <xacro:property name="servo_no_load_speed" value="14.66" />
+    <xacro:macro name="null_inertial">
+        <inertial>
+          <mass value="0.001" />
+          <inertia ixx="0.001" ixy="0" ixz="0" iyy="0.001" iyz="0" izz="0.001" />
+        </inertial>
+    </xacro:macro>
     <link name="base_link"></link>
     <joint name="baseLink_chassis" type="fixed">
@@ -188,4 +196,12 @@
         </collision>
     </link>
+    <link name="left_steering_link">
+        <xacro:null_inertial />
+    </link>
+    <joint name="left_steering_link_joint" type="fixed">
+        <parent link="chassis"/>
+        <child link="left_steering_link"/>
+        <origin xyz="0.0 0.0 0.0" rpy="0.0 0.0 0.0"/>
+    </joint>
     <link name="front_left_axle">
         <inertial>
@@ -213,4 +229,12 @@
         </collision>
     </link>
+    <link name="right_steering_link">
+        <xacro:null_inertial />
+    </link>
+    <joint name="right_steering_link_joint" type="fixed">
+        <parent link="chassis"/>
+        <child link="right_steering_link"/>
+        <origin xyz="0.0 0.0 0.0" rpy="0.0 0.0 0.0"/>
+    </joint>
     <link name="front_right_axle">
         <inertial>
@@ -246,16 +270,30 @@
         <limit lower="0.0" upper="0.0" effort="0.0" velocity="0.0"/>
     </joint> -->
-    <joint name="front_right_axle_joint" type="revolute">
+    <joint name="front_right_axle_joint" type="continuous">
         <origin xyz="1.0 -0.6 0" rpy="0 0 0" />
-        <parent link="chassis"/>
+        <parent link="right_steering_link"/>
         <child link="front_right_axle"/>
         <axis xyz="0.0 0.0 1.0"/>
         <limit lower="${-degrees_30}" upper="${degrees_30}" effort="${servo_stall_torque}" velocity="${servo_no_load_speed}" />
     </joint>
-    <joint name="front_left_axle_joint" type="revolute">
+    <joint name="front_left_axle_joint" type="continuous">
         <origin xyz="1.0 0.6 0" rpy="0 0 0" />
-        <parent link="chassis"/>
+        <parent link="left_steering_link"/>
         <child link="front_left_axle"/>
-        <axis xyz="0.0 0 1.0"/>
+        <axis xyz="0.0 0 -1.0"/>
+        <limit lower="${-degrees_30}" upper="${degrees_30}" effort="${servo_stall_torque}" velocity="${servo_no_load_speed}" />
+    </joint>
+    <joint name="front_right_wheel_joint" type="revolute">
+        <origin xyz="0.0 0.0 0" rpy="0 0 0" />
+        <parent link="front_right_axle"/>
+        <child link="front_right_wheel"/>
+        <axis xyz="0 1 0" />
+        <limit lower="${-degrees_30}" upper="${degrees_30}" effort="${servo_stall_torque}" velocity="${servo_no_load_speed}" />
+    </joint>
+    <joint name="front_left_wheel_joint" type="revolute">
+        <origin xyz="0.0 0.0 0" rpy="0 0 0" />
+        <parent link="front_left_axle"/>
+        <child link="front_left_wheel"/>
+        <axis xyz="0 1 0" />
         <limit lower="${-degrees_30}" upper="${degrees_30}" effort="${servo_stall_torque}" velocity="${servo_no_load_speed}" />
     </joint>
@@ -268,18 +306,4 @@
         <!-- <limit lower="0.0" upper="0.0" effort="0.0" velocity="0.0"/> -->
     </joint>
-    <joint name="front_right_wheel_joint" type="revolute">
-        <origin xyz="0.0 0.0 0.0" rpy="0.0 0.0 0.0"/>
-        <parent link="front_right_axle"/>
-        <child link="front_right_wheel"/>
-        <axis xyz="0 1 0" />
-        <limit lower="${-degrees_30}" upper="${degrees_30}" effort="${servo_stall_torque}" velocity="${servo_no_load_speed}" />
-    </joint>
-    <joint name="front_left_wheel_joint" type="revolute">
-        <origin xyz="0.0 0.0 0.0" rpy="0.0 0.0 0.0"/>
-        <parent link="front_left_axle"/>
-        <child link="front_left_wheel"/>
-        <axis xyz="0 1 0" />
-        <limit lower="${-degrees_30}" upper="${degrees_30}" effort="${servo_stall_torque}" velocity="${servo_no_load_speed}" />
-    </joint>
     <joint name="rear_right_wheel_joint" type="revolute">
         <origin xyz="0 -0.6 0.0" rpy="0.0 0.0 0.0"/>
